File: Schaltplan/Dreiber/Dreiber.kicad_sch (KiCad schematic)
At the start: 0 parts

Commit message: add shematic
Other:
- added sheet OpenDrainDriver1 (OpenDrainDriver.kicad_sch)
- added sheet OpenDrainDriver2 (OpenDrainDriver.kicad_sch)
- added sheet OpenDrainDriver3 (OpenDrainDriver.kicad_sch)
- added sheet ShutdownLogic (ShutdownLogic.kicad_sch)
- sheet OpenDrainDriver ports: added SENS; removed none
- sheet Versorgung ports: added VIN, VOUT; removed none
Changed lines of the file:
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@@
 (kicad_sch (version 20230121) (generator eeschema)
-  (paper "A4")
-  (sheet (at 88.9 50.8) (size 25.4 25.4) (fields_autoplaced)
-    (stroke (width 0.1524) (type solid) (color 132 0 0 1))
-    (fill (color 255 255 194 1.0000))
-    (property "Sheetname" "Versorgung" (at 88.9 50.0884 0)
-      (effects (font (size 1.27 1.27)) (justify left bottom))
-    )
-    (property "Sheetfile" "Versorgung.kicad_sch" (at 88.9 76.7846 0)
-      (effects (font (size 1.27 1.27)) (justify left top))
+  (paper "A3")
+  (wire (pts (xy 152.4 138.43) (xy 152.4 203.2))
+    (stroke (width 0) (type default))
+  )
+  (wire (pts (xy 101.6 123.19) (xy 165.1 123.19))
+    (stroke (width 0) (type default))
+  )
+  (wire (pts (xy 101.6 130.81) (xy 165.1 130.81))
+    (stroke (width 0) (type default))
+  )
+  (wire (pts (xy 152.4 203.2) (xy 215.9 203.2))
+    (stroke (width 0) (type default))
+  )
+  (wire (pts (xy 101.6 138.43) (xy 152.4 138.43))
+    (stroke (width 0) (type default))
+  )
+  (wire (pts (xy 152.4 115.57) (xy 152.4 50.8))
+    (stroke (width 0) (type default))
+  )
+  (wire (pts (xy 165.1 101.6) (xy 215.9 101.6))
+    (stroke (width 0) (type default))
+  )
+  (wire (pts (xy 101.6 115.57) (xy 152.4 115.57))
+    (stroke (width 0) (type default))
+  )
+  (wire (pts (xy 152.4 50.8) (xy 215.9 50.8))
+    (stroke (width 0) (type default))
+  )
+  (wire (pts (xy 165.1 152.4) (xy 215.9 152.4))
+    (stroke (width 0) (type default))
+  )
+  (wire (pts (xy 165.1 130.81) (xy 165.1 152.4))
+    (stroke (width 0) (type default))
+  )
+  (wire (pts (xy 165.1 123.19) (xy 165.1 101.6))
+    (stroke (width 0) (type default))
+  )
+  (sheet (at 29.21 22.86) (size 25.4 25.4) (fields_autoplaced)
+    (stroke (width 0.1524) (type solid) (color 132 0 0 1))
+    (fill (color 255 255 194 1.0000))
+    (property "Sheetname" "Versorgung" (at 29.21 22.1484 0)
+      (effects (font (size 1.27 1.27)) (justify left bottom))
+    )
+    (property "Sheetfile" "Versorgung.kicad_sch" (at 29.21 48.8446 0)
+      (effects (font (size 1.27 1.27)) (justify left top))
+    )
+    (pin "VIN" input (at 29.21 35.56 180)
+      (effects (font (size 1.27 1.27)) (justify left))
+    )
+    (pin "VOUT" input (at 54.61 35.56 0)
+      (effects (font (size 1.27 1.27)) (justify right))
     )
     (instances
@@
     )
   )
-  (sheet (at 177.8 50.8) (size 25.4 25.4) (fields_autoplaced)
-    (stroke (width 0.1524) (type solid) (color 132 0 0 1))
-    (fill (color 255 255 194 1.0000))
-    (property "Sheetname" "OpenDrainDriver" (at 177.8 50.0884 0)
-      (effects (font (size 1.27 1.27)) (justify left bottom))
-    )
-    (property "Sheetfile" "OpenDrainDriver.kicad_sch" (at 177.8 76.7846 0)
-      (effects (font (size 1.27 1.27)) (justify left top))
-    )
-    (pin "OUTPUT" input (at 203.2 63.5 0)
-      (effects (font (size 1.27 1.27)) (justify right))
-    )
-    (pin "VCC" input (at 189.23 50.8 90)
-      (effects (font (size 1.27 1.27)) (justify right))
-    )
-    (pin "INPUT" input (at 177.8 63.5 180)
-      (effects (font (size 1.27 1.27)) (justify left))
+  (sheet (at 215.9 139.7) (size 25.4 25.4) (fields_autoplaced)
+    (stroke (width 0.1524) (type solid) (color 132 0 0 1))
+    (fill (color 255 255 194 1.0000))
+    (property "Sheetname" "OpenDrainDriver2" (at 215.9 138.9884 0)
+      (effects (font (size 1.27 1.27)) (justify left bottom))
+    )
+    (property "Sheetfile" "OpenDrainDriver.kicad_sch" (at 215.9 165.6846 0)
+      (effects (font (size 1.27 1.27)) (justify left top))
+    )
+    (pin "OUTPUT" input (at 241.3 152.4 0)
+      (effects (font (size 1.27 1.27)) (justify right))
+    )
+    (pin "VCC" input (at 227.33 139.7 90)
+      (effects (font (size 1.27 1.27)) (justify right))
+    )
+    (pin "INPUT" input (at 215.9 152.4 180)
+      (effects (font (size 1.27 1.27)) (justify left))
+    )
+    (pin "SENS" input (at 241.3 158.75 0)
+      (effects (font (size 1.27 1.27)) (justify right))
+    )
+    (instances
+      (project "Dreiber"
+        (path "/b9c6537b-9919-4452-86c5-0a2d0440a6ff" (page "5"))
+      )
+    )
+  )
+  (sheet (at 74.93 101.6) (size 26.67 50.8) (fields_autoplaced)
+    (stroke (width 0.1524) (type solid) (color 132 0 0 1))
+    (fill (color 255 255 194 1.0000))
+    (property "Sheetname" "ShutdownLogic" (at 74.93 100.8884 0)
+      (effects (font (size 1.27 1.27)) (justify left bottom))
+    )
+    (property "Sheetfile" "ShutdownLogic.kicad_sch" (at 74.93 152.9846 0)
+      (effects (font (size 1.27 1.27)) (justify left top))
+    )
+    (pin "VIN" input (at 87.63 101.6 90)
+      (effects (font (size 1.27 1.27)) (justify right))
+    )
+    (pin "IN3" input (at 74.93 116.84 180)
+      (effects (font (size 1.27 1.27)) (justify left))
+    )
+    (pin "OUT3" input (at 101.6 130.81 0)
+      (effects (font (size 1.27 1.27)) (justify right))
+    )
+    (pin "IN4" input (at 74.93 121.92 180)
+      (effects (font (size 1.27 1.27)) (justify left))
+    )
+    (pin "OUT4" input (at 101.6 138.43 0)
+      (effects (font (size 1.27 1.27)) (justify right))
+    )
+    (pin "IN1" input (at 74.93 106.68 180)
+      (effects (font (size 1.27 1.27)) (justify left))
+    )
+    (pin "OUT1" input (at 101.6 115.57 0)
+      (effects (font (size 1.27 1.27)) (justify right))
+    )
+    (pin "OUT2" input (at 101.6 123.19 0)
+      (effects (font (size 1.27 1.27)) (justify right))
+    )
+    (pin "IN2" input (at 74.93 111.76 180)
+      (effects (font (size 1.27 1.27)) (justify left))
+    )
+    (pin "CCIN3" input (at 74.93 142.24 180)
+      (effects (font (size 1.27 1.27)) (justify left))
+    )
+    (pin "CCIN4" input (at 74.93 147.32 180)
+      (effects (font (size 1.27 1.27)) (justify left))
+    )
+    (pin "CCIN1" input (at 74.93 132.08 180)
+      (effects (font (size 1.27 1.27)) (justify left))
+    )
+    (pin "CCIN2" input (at 74.93 137.16 180)
+      (effects (font (size 1.27 1.27)) (justify left))
+    )
+    (instances
+      (project "Dreiber"
+        (path "/b9c6537b-9919-4452-86c5-0a2d0440a6ff" (page "7"))
+      )
+    )
+  )
+  (sheet (at 215.9 38.1) (size 25.4 25.4) (fields_autoplaced)
+    (stroke (width 0.1524) (type solid) (color 132 0 0 1))
+    (fill (color 255 255 194 1.0000))
+    (property "Sheetname" "OpenDrainDriver" (at 215.9 37.3884 0)
+      (effects (font (size 1.27 1.27)) (justify left bottom))
+    )
+    (property "Sheetfile" "OpenDrainDriver.kicad_sch" (at 215.9 64.0846 0)
+      (effects (font (size 1.27 1.27)) (justify left top))
+    )
+    (pin "OUTPUT" input (at 241.3 50.8 0)
+      (effects (font (size 1.27 1.27)) (justify right))
+    )
+    (pin "VCC" input (at 227.33 38.1 90)
+      (effects (font (size 1.27 1.27)) (justify right))
+    )
+    (pin "INPUT" input (at 215.9 50.8 180)
+      (effects (font (size 1.27 1.27)) (justify left))
+    )
+    (pin "SENS" input (at 241.3 57.15 0)
+      (effects (font (size 1.27 1.27)) (justify right))
     )
     (instances
@@
       )
     )
+  )
+  (sheet (at 215.9 88.9) (size 25.4 25.4) (fields_autoplaced)
+    (stroke (width 0.1524) (type solid) (color 132 0 0 1))
+    (fill (color 255 255 194 1.0000))
+    (property "Sheetname" "OpenDrainDriver1" (at 215.9 88.1884 0)
+      (effects (font (size 1.27 1.27)) (justify left bottom))
+    )
+    (property "Sheetfile" "OpenDrainDriver.kicad_sch" (at 215.9 114.8846 0)
+      (effects (font (size 1.27 1.27)) (justify left top))
+    )
+    (pin "OUTPUT" input (at 241.3 101.6 0)
+      (effects (font (size 1.27 1.27)) (justify right))
+    )
+    (pin "VCC" input (at 227.33 88.9 90)
+      (effects (font (size 1.27 1.27)) (justify right))
+    )
+    (pin "INPUT" input (at 215.9 101.6 180)
+      (effects (font (size 1.27 1.27)) (justify left))
+    )
+    (pin "SENS" input (at 241.3 107.95 0)
+      (effects (font (size 1.27 1.27)) (justify right))
+    )
+    (instances
+      (project "Dreiber"
+        (path "/b9c6537b-9919-4452-86c5-0a2d0440a6ff" (page "4"))
+      )
+    )
+  )
+  (sheet (at 215.9 190.5) (size 25.4 25.4) (fields_autoplaced)
+    (stroke (width 0.1524) (type solid) (color 132 0 0 1))
+    (fill (color 255 255 194 1.0000))
+    (property "Sheetname" "OpenDrainDriver3" (at 215.9 189.7884 0)
+      (effects (font (size 1.27 1.27)) (justify left bottom))
+    )
+    (property "Sheetfile" "OpenDrainDriver.kicad_sch" (at 215.9 216.4846 0)
+      (effects (font (size 1.27 1.27)) (justify left top))
+    )
+    (pin "OUTPUT" input (at 241.3 203.2 0)
+      (effects (font (size 1.27 1.27)) (justify right))
+    )
+    (pin "VCC" input (at 227.33 190.5 90)
+      (effects (font (size 1.27 1.27)) (justify right))
+    )
+    (pin "INPUT" input (at 215.9 203.2 180)
+      (effects (font (size 1.27 1.27)) (justify left))
+    )
+    (pin "SENS" input (at 241.3 209.55 0)
+      (effects (font (size 1.27 1.27)) (justify right))
+    )
+    (instances
+      (project "Dreiber"
+        (path "/b9c6537b-9919-4452-86c5-0a2d0440a6ff" (page "6"))
+      )
+    )
