File: Schaltplan/Dreiber/OpenDrainDriver.kicad_sch (KiCad schematic)
At the start: 9 parts, among them Q1 NMOS, Q2 NMOS, Q3 PMOS, U1 74AHC1G14

Commit message: add shematic
Parts:
- removed C1: C, symbol Device:C
- removed R4: R, symbol Device:R
- removed U1: 74AHC1G14, symbol 74xGxx:74AHC1G14
- added R8: 20mOhm / 3W, Resistor_SMD:R_2512_6332Metric_Pad1.40x3.35mm_HandSolder, symbol Device:R
- Q1: value NMOS -> TJ20S04M3L; footprint (none) -> Package_TO_SOT_SMD:TO-252-3_TabPin2; DigiKey (none) -> TJ20S04M3L; DigiKeyWeb (none) -> https://toshiba.semicon-storage.com/info/TJ20S04M3L_datashe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
- Q3: value PMOS -> AO3423; footprint (none) -> Package_TO_SOT_SMD:SOT-23-3; DigiKey (none) -> 785-1016-1-ND - Gurtabschnitt; DigiKeyWeb (none) -> https://www.digikey.de/de/products/detail/alpha-omega-semic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
- QFDN327N: renamed from Q2; footprint (none) -> Package_TO_SOT_SMD:SOT-23-3; DigiKey (none) -> FDN327NCT-ND; DigiKeyWeb (none) -> https://www.digikey.de/de/products/detail/onsemi/FDN327N/97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
- R1: value R -> 120R; footprint (none) -> Resistor_SMD:R_0603_1608Metric_Pad0.98x0.95mm_HandSolder
- R2: value R -> 5R; footprint (none) -> Resistor_SMD:R_0603_1608Metric_Pad0.98x0.95mm_HandSolder
- R3: value R -> 20R; footprint (none) -> Resistor_SMD:R_0603_1608Metric_Pad0.98x0.95mm_HandSolder
Connections:
- net GND: now also R8.2; no longer Q1.3 (S)
- net INPUT: now also R1.1
- new net SENS: Q1.3 (S), R8.1
Other:
- moved on the sheet: Q1, Q3, QFDN327N, R1, R2, R3
