File: Schaltplan/Dreiber/Versorgung.kicad_sch (KiCad schematic)
At the start: 12 parts, among them Q4 PMOS

Commit message: add shematic
Parts:
- removed D4: LED, symbol Device:LED
- added 2k, R13, R14: ~, Resistor_SMD:R_0201_0603Metric_Pad0.64x0.40mm_HandSolder, symbol Device:R
- added C5: 2nF, Capacitor_SMD:C_0603_1608Metric_Pad1.08x0.95mm_HandSolder, symbol Device:C
- added C6: 8,2nF, Capacitor_SMD:C_0603_1608Metric_Pad1.08x0.95mm_HandSolder, symbol Device:C
- added C7, C8: 10pF, Capacitor_SMD:C_0603_1608Metric_Pad1.08x0.95mm_HandSolder, symbol Device:C
- added D4: D_Schottky, symbol Device:D_Schottky
- added D5: 0603GBD0790S01, LED_SMD:LED_0603_1608Metric_Pad1.05x0.95mm_HandSolder, symbol Device:LED
- added L1: L, symbol Device:L
- added R10: 1k, Resistor_SMD:R_0201_0603Metric_Pad0.64x0.40mm_HandSolder, symbol Device:R
- added R9: 34k, Capacitor_SMD:C_0603_1608Metric_Pad1.08x0.95mm_HandSolder, symbol Device:R
- added U2: TPS54331, Package_SO:Diodes_SO-8EP, symbol Coildriver:TPS54331DDAR
- C2: value C_Polarized -> 100uF; footprint (none) -> Capacitor_SMD:CP_Elec_8x6.9; DigiKey (none) -> 399-A768KE107M1VLAS036CT-ND; DigiKeyWeb (none) -> https://www.digikey.de/de/products/detail/kemet/A768KE107M1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
- C3: value C -> 10pF; footprint (none) -> Capacitor_SMD:C_0603_1608Metric_Pad1.08x0.95mm_HandSolder
- C4: value C -> 100nF; footprint (none) -> Capacitor_SMD:C_0603_1608Metric_Pad1.08x0.95mm_HandSolder
- D2: value LED -> 0603RBD0700S01; footprint (none) -> LED_SMD:LED_0603_1608Metric_Pad1.05x0.95mm_HandSolder; DigiKey (none) -> 3372-0603RBD0700S01TR-ND; DigiKeyWeb (none) -> https://www.digikey.de/de/products/detail/nextgen-component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
- D3: value BZD27Cxx -> BZX585-C5V1; footprint Diode_SMD:D_SMF -> Diode_SMD:D_SOD-523; DigiKey (none) -> 1727-1659-1-ND; DigiKeyWeb (none) -> https://www.digikey.de/de/products/detail/nexperia-usa-inc/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
- F1: value Fuse -> 100mA; footprint (none) -> Fuse:Fuse_0402_1005Metric_Pad0.77x0.64mm_HandSolder; DigiKey (none) -> 478-6485-1-ND; DigiKeyWeb (none) -> https://www.digikey.de/de/products/detail/kyocera-avx/F0402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
- Q4: value PMOS -> PMV250EPEA; footprint (none) -> Package_TO_SOT_SMD:SOT-23; DigiKey (none) -> 1727-2303-1-ND; DigiKey-Web (none) -> https://www.digikey.de/de/products/detail/nexperia-usa-inc/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
- R5: value R -> 2k7; footprint (none) -> Resistor_SMD:R_0603_1608Metric_Pad0.98x0.95mm_HandSolder
- R6: value R -> 23k; footprint (none) -> Resistor_SMD:R_0201_0603Metric_Pad0.64x0.40mm_HandSolder
- R7: value R -> 10k2; footprint (none) -> Resistor_SMD:R_0201_0603Metric_Pad0.64x0.40mm_HandSolder
Connections:
- net GND: now also C4.2, 2k.2, C5.2, C6.2, C8.2, D4.2 (A), D5.1 (K), R13.2, U2.7 (GND), U2.9 (PowerPad)
- net VOUT: now reaches R7.1
- net VOUT: now also C8.1, L1.2, R10.1
- net at R7.2: now also 2k.1, U2.5 (VSENSE)
- net VIN: now reaches D1.2 (A2), F1.1, R5.1
- net at C4.1: now also C2.1, D3.1 (K), Q4.3 (S), R14.1, U2.2 (VIN)
- new net: C5.1, R9.2
- new net: C7.2, D4.1 (K), L1.1, U2.8 (PH)
- new net: C6.1, R9.1, U2.6 (COMP)
- new net: R13.1, R14.2, U2.3 (EN)
- new net: D5.2 (A), R10.2
- new net: C7.1, U2.1 (BOOT)
- new net: C3.1, U2.4 (SS)
Other:
- note added: "Grün"
- note added: "Noch machen"
- note added: "Rot"
- note added: "Versorgung"
- moved on the sheet: C2, C4, D1, D2, D3, F1, Q4, R5, R6
